Commit message: modified erp42_teleop, erp42_vehicle

File: erp42_vehicle/erp42_vehicle_description/urdf/erp42_vehicle.urdf.xacro (robot description, xacro)
@@ -141,5 +141,5 @@
             <!-- VLP-16 -->
   <VLP-16 parent="base_link" name="velodyne" topic="/velodyne_points" hz="50" samples="1024" gpu="false" lasers="16" max_range="100">
-    <origin xyz="0 0 0.1" rpy="0 0 0" />
+    <origin xyz="0 0 0.3" rpy="0 0 0" />
   </VLP-16>
     <!-- IMU link -->
@@ -155,5 +155,5 @@
   <joint name="camera_joint" type="fixed">
     <axis xyz="0 1 0" />
-    <origin xyz="0 0 0.3" rpy="0 0.1 0"/>
+    <origin xyz="0.20 0 0.5" rpy="0 -0.1 0"/>
     <parent link="base_link"/>
     <child link="camera_link"/>
@@ -162,10 +162,10 @@
   <xacro:property name="camera_size" value="0.05" /> <!-- Size of square 'camera' box -->
   <link name="camera_link">
-  <collision>
+<!--  <collision>
       <geometry>
           <box size=".1 .3 .1"/>
       </geometry>
       <contact_coefficients mu="0" kp="1000.0" kd="1.0"/>
-  </collision>
+  </collision>-->
     <visual>
         <geometry>
@@ -188,5 +188,5 @@
       <update_rate>30.0</update_rate>
       <camera name="head">
-        <horizontal_fov>1.5</horizontal_fov>
+        <horizontal_fov>1.047</horizontal_fov>
         <image>
           <width>600</width>
@@ -195,6 +195,6 @@
         </image>
         <clip>
-          <near>0.02</near>
-          <far>300</far>
+          <near>0.1</near>
+          <far>100</far>
         </clip>
         <noise>
@@ -209,5 +209,5 @@
       <plugin name="camera_controller" filename="libgazebo_ros_openni_kinect.so">
         <alwaysOn>true</alwaysOn>
-        <updateRate>0.0</updateRate>
+        <updateRate>10.0</updateRate>
         <cameraName>camera_ir</cameraName>
         <imageTopicName>/camera/color/image_raw</imageTopicName>
@@ -217,5 +217,5 @@
         <pointCloudTopicName>/camera/depth/points</pointCloudTopicName>
         <frameName>camera_link</frameName>
-        <pointCloudCutoff>0.5</pointCloudCutoff>
+        <pointCloudCutoff>0.4</pointCloudCutoff>
         <pointCloudCutoffMax>3.0</pointCloudCutoffMax>
         <distortionK1>0.0</distortionK1>
@@ -228,5 +228,5 @@
         <Cy>0</Cy>
         <focalLength>0</focalLength>
-        <hackBaseline>0</hackBaseline>
+        <hackBaseline>0.07</hackBaseline>
       </plugin>
     </sensor>

File: erp42_vehicle/erp42_vehicle_description/urdf/wheel.xacro (robot description, xacro)
@@ -118,5 +118,5 @@
           <cylinder radius="${wheel_radius}" length="${wheel_thickness}"/>
         </geometry>
-        <material name="red" />
+        <material name="black" />
       </visual>
       <collision>

Commit message: update erp42_slam_3d

File: erp42_vehicle/erp42_vehicle_description/urdf/erp42_vehicle.urdf.xacro (robot description, xacro)
@@ -145,5 +145,5 @@
     <!-- IMU link -->
    <joint name="imu_joint" type="fixed">
-    <axis xyz="0 1 0" />
+    <axis xyz="0 0 1" />
     <origin xyz="0 0 0.02" rpy="0 0 0"/>
     <parent link="base_link"/>
